File: hardware/sample_project.kicad_pcb (KiCad board)
At the start: 2 copper layers, 43.2 x 43.2 mm, 8 parts

Commit message: added some misc info
Parts:
- added JP1: SolderJumper_2_Open, Jumper:SolderJumper-2_P1.3mm_Open_TrianglePad1.0x1.5mm, F.Cu at (134.5, 123.2)
- added TP1: TestPoint, TestPoint:TestPoint_Keystone_5015_Micro_Mini, F.Cu at (134.5, 119.2)

Commit message: added test points
Connections:
- H1 pad 1: unconnected-(H1-Pad1) -> GND
- JP1 pad 1: unconnected-(JP1-A-Pad1) -> MCU_SCLK
- JP1 pad 2: unconnected-(JP1-B-Pad2) -> /Holes and fiducials/SCLK
